File: Hardware/Photon_I2C_Shield.sch (EAGLE design)
At the start: 21 parts

Commit message: Finishing touches before going live.
Other:
- note added: "Joel Bartlett"
Changed lines of the file:
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@@
 <wire x1="248.92" y1="129.54" x2="147.32" y2="129.54" width="0.2032" layer="97" style="shortdash"/>
 <text x="182.88" y="175.26" size="1.778" layer="97" font="vector">VCC Range: 1.9v-3.6v</text>
+<text x="170.688" y="11.43" size="2.54" layer="94">Joel Bartlett</text>
 </plain>
 <instances>
