File: Panel/Photon_I2C_Shield_Panel.brd (EAGLE design)
At the start: 171.7 x 171.6 mm, 252 parts

Commit message: New panel with Qwiic silk.
Parts:
- removed H25, H26, H27, H28, H29, H30, H31, H32, H33, H34, H35, H36, H37, H38, H39, H40, H41, H42, H43, H44, H45, H46, H47, H48: STAND-OFF, SparkFun-Hardware:STAND-OFF
- removed J25, J26, J27, J28, J29, J30, J31, J32, J33, J34, J35, J36, J37, J38, J39, J40, J41, J42, J43, J44, J45, J46, J47, J48: (no value), SparkX:1X04_1MM_RA
- removed JP100, JP107, JP108, JP109, JP110, JP117, JP118, JP119, JP120, JP67, JP68, JP69, JP70, JP77, JP78, JP79, JP80, JP87, JP88, JP89, JP90, JP97, JP98, JP99: (no value), SparkFun-Connectors:1X09_NO_SILK
- removed JP101, JP111, JP61, JP71, JP81, JP91: PARTICLE_PHOTONTEMPLATE_NO_STANDOFF, SparkFun-Boards:PARTICLE_PHOTON_TEMPLATE_NO_STANDOFF
- removed JP102, JP112, JP62, JP72, JP82, JP92: (no value), SparkFun-Connectors:1X04
- removed JP103, JP104, JP113, JP114, JP63, JP64, JP73, JP74, JP83, JP84, JP93, JP94: (no value), SparkFun-Connectors:1X03
- removed JP105, JP106, JP115, JP116, JP65, JP66, JP75, JP76, JP85, JP86, JP95, JP96: (no value), SparkFun-Connectors:1X10_NO_SILK
- removed LOGO10, LOGO11, LOGO12, LOGO7, LOGO8, LOGO9: OSHW-LOGOM, SparkFun-Aesthetics:OSHW-LOGO-M
- removed U$13, U$15, U$17, U$19, U$21, U$23: (no value), SparkX:SPARKX-TINY
- removed U$14, U$16, U$18, U$20, U$22, U$24: SPARKX-LOGO5, SparkX:SPARKX-LARGE
Connections:
- removed net A36: JP61.7, JP61.A5
- removed net A37: JP61.8, JP61.A4
- removed net A38: JP61.9, JP61.A3
- removed net A39: JP61.10, JP61.A2
- removed net A40: JP61.11, JP61.A1
- removed net A41: JP61.12, JP61.A0
- removed net A42: JP71.7, JP71.A5
- removed net A43: JP71.8, JP71.A4
- removed net A44: JP71.9, JP71.A3
- removed net A45: JP71.10, JP71.A2
- removed net A46: JP71.11, JP71.A1
- removed net A47: JP71.12, JP71.A0
- removed net A48: JP81.7, JP81.A5
- removed net A49: JP81.8, JP81.A4
- removed net A50: JP81.9, JP81.A3
- removed net A51: JP81.10, JP81.A2
- removed net A52: JP81.11, JP81.A1
- removed net A53: JP81.12, JP81.A0
- removed net A54: JP91.7, JP91.A5
- removed net A55: JP91.8, JP91.A4
- removed net A56: JP91.9, JP91.A3
- removed net A57: JP91.10, JP91.A2
- removed net A58: JP91.11, JP91.A1
- removed net A59: JP91.12, JP91.A0
- removed net A60: JP101.7, JP101.A5
- removed net A61: JP101.8, JP101.A4
- removed net A62: JP101.9, JP101.A3
- removed net A63: JP101.10, JP101.A2
- removed net A64: JP101.11, JP101.A1
- removed net A65: JP101.12, JP101.A0
- removed net A66: JP111.7, JP111.A5
- removed net A67: JP111.8, JP111.A4
- removed net A68: JP111.9, JP111.A3
- removed net A69: JP111.10, JP111.A2
- removed net A70: JP111.11, JP111.A1
- removed net A71: JP111.12, JP111.A0
- removed net D37: JP61.20, JP61.D7
- removed net D38: JP61.19, JP61.D6
- removed net D39: JP61.18, JP61.D5
- removed net D40: JP61.17, JP61.D4
- removed net D41: JP61.16, JP61.D3
- removed net D42: JP61.15, JP61.D2
- removed net D43: JP71.20, JP71.D7
- removed net D44: JP71.19, JP71.D6
- removed net D45: JP71.18, JP71.D5
- removed net D46: JP71.17, JP71.D4
- removed net D47: JP71.16, JP71.D3
- removed net D48: JP71.15, JP71.D2
- removed net D49: JP81.20, JP81.D7
- removed net D50: JP81.19, JP81.D6
- removed net D51: JP81.18, JP81.D5
- removed net D52: JP81.17, JP81.D4
- removed net D53: JP81.16, JP81.D3
- removed net D54: JP81.15, JP81.D2
- removed net D55: JP91.20, JP91.D7
- removed net D56: JP91.19, JP91.D6
- removed net D57: JP91.18, JP91.D5
- removed net D58: JP91.17, JP91.D4
- removed net D59: JP91.16, JP91.D3
- removed net D60: JP91.15, JP91.D2
- removed net D61: JP101.20, JP101.D7
- removed net D62: JP101.19, JP101.D6
- removed net D63: JP101.18, JP101.D5
- removed net D64: JP101.17, JP101.D4
- removed net D65: JP101.16, JP101.D3
- removed net D66: JP101.15, JP101.D2
- removed net D67: JP111.20, JP111.D7
- removed net D68: JP111.19, JP111.D6
- removed net D69: JP111.18, JP111.D5
- removed net D70: JP111.17, JP111.D4
- removed net D71: JP111.16, JP111.D3
- removed net D72: JP111.15, JP111.D2
- removed net DAC10: JP101.6, JP101.DAC
- removed net DAC11: JP111.6, JP111.DAC
- removed net DAC6: JP61.6, JP61.DAC
- removed net DAC7: JP71.6, JP71.DAC
- removed net DAC8: JP81.6, JP81.DAC
- removed net DAC9: JP91.6, JP91.DAC
- removed net GND10: J41.1, J42.1, J43.1, J44.1, JP101.2, JP101.21, JP101.GND@0, JP101.GND@2, JP102.1, JP104.1, JP104.2, JP104.3
- removed net GND11: J45.1, J46.1, J47.1, J48.1, JP111.2, JP111.21, JP111.GND@0, JP111.GND@2, JP112.1, JP114.1, JP114.2, JP114.3
- removed net GND6: J25.1, J26.1, J27.1, J28.1, JP61.2, JP61.21, JP61.GND@0, JP61.GND@2, JP62.1, JP64.1, JP64.2, JP64.3
- removed net GND7: J29.1, J30.1, J31.1, J32.1, JP71.2, JP71.21, JP71.GND@0, JP71.GND@2, JP72.1, JP74.1, JP74.2, JP74.3
- removed net GND8: J33.1, J34.1, J35.1, J36.1, JP81.2, JP81.21, JP81.GND@0, JP81.GND@2, JP82.1, JP84.1, JP84.2, JP84.3
- removed net GND9: J37.1, J38.1, J39.1, J40.1, JP91.2, JP91.21, JP91.GND@0, JP91.GND@2, JP92.1, JP94.1, JP94.2, JP94.3
- removed net RST10: JP101.23, JP101.RST
- removed net RST11: JP111.23, JP111.RST
- removed net RST6: JP61.23, JP61.RST
- removed net RST7: JP71.23, JP71.RST
- removed net RST8: JP81.23, JP81.RST
- removed net RST9: JP91.23, JP91.RST
- removed net RX10: JP101.4, JP101.RX
- removed net RX11: JP111.4, JP111.RX
- removed net RX6: JP61.4, JP61.RX
- removed net RX7: JP71.4, JP71.RX
- removed net RX8: JP81.4, JP81.RX
- removed net RX9: JP91.4, JP91.RX
- removed net SCL10: J41.4, J42.4, J43.4, J44.4, JP101.14, JP101.D1, JP102.4
- removed net SCL11: J45.4, J46.4, J47.4, J48.4, JP111.14, JP111.D1, JP112.4
- removed net SCL6: J25.4, J26.4, J27.4, J28.4, JP61.14, JP61.D1, JP62.4
- removed net SCL7: J29.4, J30.4, J31.4, J32.4, JP71.14, JP71.D1, JP72.4
- removed net SCL8: J33.4, J34.4, J35.4, J36.4, JP81.14, JP81.D1, JP82.4
- removed net SCL9: J37.4, J38.4, J39.4, J40.4, JP91.14, JP91.D1, JP92.4
- removed net SDA10: J41.3, J42.3, J43.3, J44.3, JP101.13, JP101.D0, JP102.3
- removed net SDA11: J45.3, J46.3, J47.3, J48.3, JP111.13, JP111.D0, JP112.3
- removed net SDA6: J25.3, J26.3, J27.3, J28.3, JP61.13, JP61.D0, JP62.3
- removed net SDA7: J29.3, J30.3, J31.3, J32.3, JP71.13, JP71.D0, JP72.3
- removed net SDA8: J33.3, J34.3, J35.3, J36.3, JP81.13, JP81.D0, JP82.3
- removed net SDA9: J37.3, J38.3, J39.3, J40.3, JP91.13, JP91.D0, JP92.3
- removed net TX10: JP101.3, JP101.TX
- removed net TX11: JP111.3, JP111.TX
- removed net TX6: JP61.3, JP61.TX
- removed net TX7: JP71.3, JP71.TX
- removed net TX8: JP81.3, JP81.TX
- removed net TX9: JP91.3, JP91.TX
- removed net VBAT10: JP101.22, JP101.VBAT
- removed net VBAT11: JP111.22, JP111.VBAT
- removed net VBAT6: JP61.22, JP61.VBAT
- removed net VBAT7: JP71.22, JP71.VBAT
- removed net VBAT8: JP81.22, JP81.VBAT
- removed net VBAT9: JP91.22, JP91.VBAT
- removed net VCC10: J41.2, J42.2, J43.2, J44.2, JP101.24, JP101.3V3, JP102.2, JP103.1, JP103.2, JP103.3
- removed net VCC11: J45.2, J46.2, J47.2, J48.2, JP111.24, JP111.3V3, JP112.2, JP113.1, JP113.2, JP113.3
- removed net VCC6: J25.2, J26.2, J27.2, J28.2, JP61.24, JP61.3V3, JP62.2, JP63.1, JP63.2, JP63.3
- removed net VCC7: J29.2, J30.2, J31.2, J32.2, JP71.24, JP71.3V3, JP72.2, JP73.1, JP73.2, JP73.3
- removed net VCC8: J33.2, J34.2, J35.2, J36.2, JP81.24, JP81.3V3, JP82.2, JP83.1, JP83.2, JP83.3
- removed net VCC9: J37.2, J38.2, J39.2, J40.2, JP91.24, JP91.3V3, JP92.2, JP93.1, JP93.2, JP93.3
- removed net VIN10: JP101.1, JP101.VIN
- removed net VIN11: JP111.1, JP111.VIN
- removed net VIN6: JP61.1, JP61.VIN
- removed net VIN7: JP71.1, JP71.VIN
- removed net VIN8: JP81.1, JP81.VIN
- removed net VIN9: JP91.1, JP91.VIN
- removed net WKP10: JP101.5, JP101.WKP
- removed net WKP11: JP111.5, JP111.WKP
- removed net WKP6: JP61.5, JP61.WKP
- removed net WKP7: JP71.5, JP71.WKP
- removed net WKP8: JP81.5, JP81.WKP
- removed net WKP9: JP91.5, JP91.WKP
Routing:
- net SDA9: track 95.3 -> 0.00 mm, vias 2 -> 0
- net SDA6: track 95.3 -> 0.00 mm, vias 2 -> 0
- net SDA8: track 95.3 -> 0.00 mm, vias 2 -> 0
- net SDA7: track 95.3 -> 0.00 mm, vias 2 -> 0
- net SDA11: track 95.3 -> 0.00 mm, vias 2 -> 0
- net SDA10: track 95.3 -> 0.00 mm, vias 2 -> 0
- net SCL9: track 88.9 -> 0.00 mm, vias 3 -> 0
- net SCL8: track 88.9 -> 0.00 mm, vias 3 -> 0
- net SCL7: track 88.9 -> 0.00 mm, vias 3 -> 0
- net SCL6: track 88.9 -> 0.00 mm, vias 3 -> 0
- net SCL11: track 88.9 -> 0.00 mm, vias 3 -> 0
- net SCL10: track 88.9 -> 0.00 mm, vias 3 -> 0
- net VCC7: track 81.7 -> 0.00 mm, vias 1 -> 0
- net VCC11: track 81.7 -> 0.00 mm, vias 1 -> 0
- net VCC10: track 81.7 -> 0.00 mm, vias 1 -> 0
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- removed copper zone on layer 1, net GND10
- removed copper zone on layer 16, net GND10
- removed copper zone on layer 1, net GND11
- removed copper zone on layer 16, net GND11
- removed copper zone on layer 1, net GND6
- removed copper zone on layer 16, net GND6
- removed copper zone on layer 1, net GND7
- removed copper zone on layer 16, net GND7
- removed copper zone on layer 1, net GND8
- removed copper zone on layer 16, net GND8
- removed copper zone on layer 1, net GND9
- removed copper zone on layer 16, net GND9
Other:
- board size 171.7 x 171.6 mm -> 147.2 x 83.4 mm
- board text added: "Photon Qwiic Shield"
- board text added: "mill out"
- board text added: "v-score"
- board text removed: "Adding frame around panel is acceptable"
- board text removed: "Photon I2C Shield"
- board text removed: "VScore"
